Commit message: - Fix sampling script by dumping the buffer using rostopic echo - Change color from white to yellow - Remove unused gravity tag
Signed-off-by: Timo Korthals <tkorthals@cit-ec.uni-bielefeld.de>

File: catkin_ws/src/rubiks_description/urdf/camera.xacro (robot description, xacro)
@@ -49,4 +49,5 @@
   <gazebo reference="${name}">
     <sensor type="camera" name="camera1">
+      <always_on>0</always_on>
       <update_rate>20.0</update_rate>
       <camera name="head">
@@ -71,5 +72,7 @@
       </camera>
       <plugin name="camera_controller" filename="libgazebo_ros_camera.so">
+      <!-- plugin name="camera_controller" filename="libgazebo_ros_triggered_camera.so" -->
         <robotNamespace></robotNamespace>
+        <!-- triggerTopicName>image_trigger</triggerTopicName -->
         <alwaysOn>true</alwaysOn>
         <updateRate>0.0</updateRate>
@@ -92,6 +95,4 @@
     <static>true</static>
     <self_collide>0</self_collide>
-    <kinematic>0</kinematic>
-    <gravity>0</gravity>
 </gazebo>
 </robot>

File: catkin_ws/src/rubiks_description/urdf/rubiks_cube_no_mesh.xacro (robot description, xacro)
@@ -53,5 +53,5 @@
           <box size="0.1 0.1 0.001"/>
         </geometry>
-        <material name="white"/>
+        <material name="yellow"/>
     </visual>
     <inertial>
