Commit message: - Add Rubik's cube to Gazebo and rviz - Various refinements in the cube model definition - Add slides
Signed-off-by: Timo Korthals <tkorthals@cit-ec.uni-bielefeld.de>

File: catkin_ws/src/rubiks_description/urdf/rubiks_cube_no_mesh.xacro (robot description, xacro)
@@ -5,11 +5,15 @@
   <!-- Import Gazebo elements, including Gazebo colors -->
   <xacro:include filename="$(find rubiks_description)/urdf/rubiks_cube.gazebo" />
+  <xacro:property name="world_cube_x" value="$(arg world_cube_x)"/>
+  <xacro:property name="world_cube_y" value="$(arg world_cube_y)"/>
+  <xacro:property name="world_cube_z" value="$(arg world_cube_z)"/>
   <link name="world"/>
   <joint name="fixed" type="fixed">
     <parent link="world"/>
-    <child link="base_link"/>
+    <child link="base_link_cube"/>
+    <origin xyz="$(arg world_cube_x) $(arg world_cube_y) $(arg world_cube_z)" rpy="0 0 0"/>
   </joint>
   <!-- Base Link -->
-  <link name="base_link">
+  <link name="base_link_cube">
     <collision>
       <origin xyz="0.0 0.0 0.0" rpy="0.0 0.0 0.0"/>
@@ -35,5 +39,5 @@
   </link>
   <joint name="bot_joint" type="fixed">
-    <parent link="base_link"/>
+    <parent link="base_link_cube"/>
     <child link="bot_link"/>
     <origin xyz="0 0 -0.05" rpy="0 0 0"/>
@@ -65,5 +69,5 @@
   </link>
 <joint name="top_joint" type="fixed">
-    <parent link="base_link"/>
+    <parent link="base_link_cube"/>
     <child link="top_link"/>
     <origin xyz="0 0 0.05" rpy="0 0 0"/>
@@ -95,5 +99,5 @@
   </link>
 <joint name="left_joint" type="fixed">
-    <parent link="base_link"/>
+    <parent link="base_link_cube"/>
     <child link="left_link"/>
     <origin xyz="0 0.05 0.0" rpy="0 0 0"/>
@@ -125,5 +129,5 @@
   </link>
   <joint name="right_joint" type="fixed">
-    <parent link="base_link"/>
+    <parent link="base_link_cube"/>
     <child link="right_link"/>
     <origin xyz="0 -0.05 0.0" rpy="0 0 0"/>
@@ -155,5 +159,5 @@
   </link>
 <joint name="front_joint" type="fixed">
-    <parent link="base_link"/>
+    <parent link="base_link_cube"/>
     <child link="front_link"/>
     <origin xyz="0.05 0.0 0.0" rpy="0 0 0"/>
@@ -185,5 +189,5 @@
   </link>
   <joint name="back_joint" type="fixed">
-    <parent link="base_link"/>
+    <parent link="base_link_cube"/>
     <child link="back_link"/>
     <origin xyz="-0.05 0.0 0.0" rpy="0 0 0"/>

Commit message: Add final Rubik's cube of edge size 4.5 cm
Signed-off-by: Timo Korthals <tkorthals@cit-ec.uni-bielefeld.de>

File: catkin_ws/src/rubiks_description/urdf/rubiks_cube_no_mesh.xacro (robot description, xacro)
@@ -8,4 +8,5 @@
   <xacro:property name="world_cube_y" value="$(arg world_cube_y)"/>
   <xacro:property name="world_cube_z" value="$(arg world_cube_z)"/>
+  <xacro:property name="cube_size" value="$(arg cube_size)"/>
   <link name="world"/>
   <joint name="fixed" type="fixed">
@@ -25,5 +26,5 @@
         <origin xyz="0.0 0.0 0.0" rpy="0.0 0.0 0.0"/>
         <geometry>
-          <!-- mesh filename="package://rubiks_description/meshes/rubiks_cube/cube.dae" scale="0.1 0.1 0.1"/ -->
+          <!-- mesh filename="package://rubiks_description/meshes/rubiks_cube/cube.dae" scale="${cube_size} ${cube_size} ${cube_size}"/ -->
           <box size="0.01 0.01 0.01"/>
         </geometry>
@@ -41,5 +42,5 @@
     <parent link="base_link_cube"/>
     <child link="bot_link"/>
-    <origin xyz="0 0 -0.05" rpy="0 0 0"/>
+    <origin xyz="0 0 -${cube_size / 2.0}" rpy="0 0 0"/>
     <axis xyz="1 1 1"/>
     <dynamics damping="0.0"/>
@@ -49,11 +50,11 @@
       <origin xyz="0.0 0.0 0.0" rpy="0.0 0.0 0.0"/>
       <geometry>
-        <box size="0.1 0.1 0.001"/>
-      </geometry>
-    </collision>
-    <visual>
-        <origin xyz="0.0 0.0 0.0" rpy="0.0 0.0 0.0"/>
-        <geometry>
-          <box size="0.1 0.1 0.001"/>
+        <box size="${cube_size} ${cube_size} 0.001"/>
+      </geometry>
+    </collision>
+    <visual>
+        <origin xyz="0.0 0.0 0.0" rpy="0.0 0.0 0.0"/>
+        <geometry>
+          <box size="${cube_size} ${cube_size} 0.001"/>
         </geometry>
         <material name="yellow"/>
@@ -71,5 +72,5 @@
     <parent link="base_link_cube"/>
     <child link="top_link"/>
-    <origin xyz="0 0 0.05" rpy="0 0 0"/>
+    <origin xyz="0 0 ${cube_size / 2.0}" rpy="0 0 0"/>
     <axis xyz="1 1 1"/>
     <dynamics damping="0.0"/>
@@ -79,11 +80,11 @@
       <origin xyz="0.0 0.0 0.0" rpy="0.0 0.0 0.0"/>
       <geometry>
-        <box size="0.1 0.1 0.001"/>
-      </geometry>
-    </collision>
-    <visual>
-        <origin xyz="0.0 0.0 0.0" rpy="0.0 0.0 0.0"/>
-        <geometry>
-          <box size="0.1 0.1 0.001"/>
+        <box size="${cube_size} ${cube_size} 0.001"/>
+      </geometry>
+    </collision>
+    <visual>
+        <origin xyz="0.0 0.0 0.0" rpy="0.0 0.0 0.0"/>
+        <geometry>
+          <box size="${cube_size} ${cube_size} 0.001"/>
         </geometry>
         <material name="green"/>
@@ -101,5 +102,5 @@
     <parent link="base_link_cube"/>
     <child link="left_link"/>
-    <origin xyz="0 0.05 0.0" rpy="0 0 0"/>
+    <origin xyz="0 ${cube_size / 2.0} 0.0" rpy="0 0 0"/>
     <axis xyz="1 1 1"/>
     <dynamics damping="0.0"/>
@@ -109,11 +110,11 @@
       <origin xyz="0.0 0.0 0.0" rpy="0.0 0.0 0.0"/>
       <geometry>
-        <box size="0.1 0.001 0.1"/>
-      </geometry>
-    </collision>
-    <visual>
-        <origin xyz="0.0 0.0 0.0" rpy="0.0 0.0 0.0"/>
-        <geometry>
-          <box size="0.1 0.001 0.1"/>
+        <box size="${cube_size} 0.001 ${cube_size}"/>
+      </geometry>
+    </collision>
+    <visual>
+        <origin xyz="0.0 0.0 0.0" rpy="0.0 0.0 0.0"/>
+        <geometry>
+          <box size="${cube_size} 0.001 ${cube_size}"/>
         </geometry>
         <material name="red"/>
@@ -131,5 +132,5 @@
     <parent link="base_link_cube"/>
     <child link="right_link"/>
-    <origin xyz="0 -0.05 0.0" rpy="0 0 0"/>
+    <origin xyz="0 -${cube_size / 2.0} 0.0" rpy="0 0 0"/>
     <axis xyz="1 1 1"/>
     <dynamics damping="0.0"/>
@@ -139,11 +140,11 @@
       <origin xyz="0.0 0.0 0.0" rpy="0.0 0.0 0.0"/>
       <geometry>
-        <box size="0.1 0.001 0.1"/>
-      </geometry>
-    </collision>
-    <visual>
-        <origin xyz="0.0 0.0 0.0" rpy="0.0 0.0 0.0"/>
-        <geometry>
-          <box size="0.1 0.001 0.1"/>
+        <box size="${cube_size} 0.001 ${cube_size}"/>
+      </geometry>
+    </collision>
+    <visual>
+        <origin xyz="0.0 0.0 0.0" rpy="0.0 0.0 0.0"/>
+        <geometry>
+          <box size="${cube_size} 0.001 ${cube_size}"/>
         </geometry>
         <material name="purple"/>
@@ -161,5 +162,5 @@
     <parent link="base_link_cube"/>
     <child link="front_link"/>
-    <origin xyz="0.05 0.0 0.0" rpy="0 0 0"/>
+    <origin xyz="${cube_size / 2.0} 0.0 0.0" rpy="0 0 0"/>
     <axis xyz="1 1 1"/>
     <dynamics damping="0.0"/>
@@ -169,11 +170,11 @@
       <origin xyz="0.0 0.0 0.0" rpy="0.0 0.0 0.0"/>
       <geometry>
-        <box size="0.001 0.1 0.1"/>
-      </geometry>
-    </collision>
-    <visual>
-        <origin xyz="0.0 0.0 0.0" rpy="0.0 0.0 0.0"/>
-        <geometry>
-          <box size="0.001 0.1 0.1"/>
+        <box size="0.001 ${cube_size} ${cube_size}"/>
+      </geometry>
+    </collision>
+    <visual>
+        <origin xyz="0.0 0.0 0.0" rpy="0.0 0.0 0.0"/>
+        <geometry>
+          <box size="0.001 ${cube_size} ${cube_size}"/>
         </geometry>
         <material name="blue"/>
@@ -191,5 +192,5 @@
     <parent link="base_link_cube"/>
     <child link="back_link"/>
-    <origin xyz="-0.05 0.0 0.0" rpy="0 0 0"/>
+    <origin xyz="-${cube_size / 2.0} 0.0 0.0" rpy="0 0 0"/>
     <axis xyz="1 1 1"/>
     <dynamics damping="0.0"/>
@@ -199,11 +200,11 @@
       <origin xyz="0.0 0.0 0.0" rpy="0.0 0.0 0.0"/>
       <geometry>
-        <box size="0.001 0.1 0.1"/>
-      </geometry>
-    </collision>
-    <visual>
-        <origin xyz="0.0 0.0 0.0" rpy="0.0 0.0 0.0"/>
-        <geometry>
-          <box size="0.001 0.1 0.1"/>
+        <box size="0.001 ${cube_size} ${cube_size}"/>
+      </geometry>
+    </collision>
+    <visual>
+        <origin xyz="0.0 0.0 0.0" rpy="0.0 0.0 0.0"/>
+        <geometry>
+          <box size="0.001 ${cube_size} ${cube_size}"/>
         </geometry>
         <material name="orange"/>
